File: hardware/noise-o-meter.sch (KiCad schematic (older format))
At the start: 39 parts, among them J1 USB_B_Micro, U1 NCP1117-3.3_SOT223, U2 RP2040

Commit message: Update schema
Parts:
- added C14, C16: 100n, symbol Device:C
- added C15: 10n, symbol Device:C
- added C17, C?: 10u, symbol Device:C
- added C18: 100p, symbol Device:C
- added C19, C20: 27p, symbol Device:C
- added J2: Conn_01x02, symbol Connector_Generic:Conn_01x02
- added J? (x2): Conn_02x18_Odd_Even, symbol Connector_Generic:Conn_02x18_Odd_Even
- added R12, R14, R15, R18, R20: 1k, symbol Device:R
- added R13: DNF, symbol Device:R
- added R16, R17: 1m, symbol Device:R
- added R19: 22k, symbol Device:R
- added RV1: R_POT, symbol Device:R_POT
- added U3: W25Q80DVSNIG, symbol Memory_Flash:W25Q80DVSNIG
- added Y1: Crystal, symbol Device:Crystal
- gave numbers to parts that had none: 3
Connections:
- net labels added: +3V3, MIC_OUT, SWCLK, SWD, ~USB_BOOT
- net labels removed: +3.3V, XIN, XOUT
- wire segments 178 -> 367
Other:
- moved on the sheet: C4, C5, D1, D2, D3, D4, D5, D6, D7, D8, D9, J1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

Commit message: Adjust
Parts:
- gave numbers to parts that had none: 3
Connections:
- wire segments 367 -> 368
- no-connect marks 0 -> 1
Other:
- note added: "Flash"
- note added: "IO headers"
- note added: "LEDs\n"
- note added: "Make sure C3 is close to pin 45 of the RP2040"
- note added: "Make sure C6 is close to pin 44 of RP2040\n"
- note added: "Make sure R1 and R2 are close to RP2040\n"
- note added: "Microphone"
- note added: "Power"
- note added: "RP2040\n"
- moved on the sheet: C1, C10, C11, C12, C13, C14, C15, C16, C17, C18, C19, C2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

Commit message: Fix debug probe
Parts:
- removed J3: 640456-2, digikey-footprints:PinHeader_1x2_P2.54mm_Drill1.02mm, symbol dk_Rectangular-Connectors-Headers-Male-Pins:640456-2
- added J?: Conn_01x04, symbol Connector_Generic:Conn_01x04
Connections:
- wire segments 368 -> 372
Changed lines of the file:
@@
 	5100 5350 5200 5350
-Wire Wire Line
-	5100 5250 5200 5250
 Wire Wire Line
 	5100 5050 5200 5050
@@
 	1    13950 7700
 	1    0    0    -1
-$EndComp
-$Comp
-L dk_Rectangular-Connectors-Headers-Male-Pins:640456-2 J3
-U 1 1 61674BE8
-P 1900 5100
-F 0 "J3" V 1675 5108 50  0000 C CNN
-F 1 "640456-2" V 1766 5108 50  0000 C CNN
-F 2 "digikey-footprints:PinHeader_1x2_P2.54mm_Drill1.02mm" H 2100 5300 60  0001 L CNN
-F 3 "https://www.te.com/commerce/DocumentDelivery/DDEController?Action=srchrtrv&DocNm=640456&DocType=Customer+Drawing&DocLang=English" H 2100 5400 60  0001 L CNN
-F 4 "A1921-ND" H 2100 5500 60  0001 L CNN "Digi-Key_PN"
-F 5 "640456-2" H 2100 5600 60  0001 L CNN "MPN"
-F 6 "Connectors, Interconnects" H 2100 5700 60  0001 L CNN "Category"
-F 7 "Rectangular Connectors - Headers, Male Pins" H 2100 5800 60  0001 L CNN "Family"
-F 8 "https://www.te.com/commerce/DocumentDelivery/DDEController?Action=srchrtrv&DocNm=640456&DocType=Customer+Drawing&DocLang=English" H 2100 5900 60  0001 L CNN "DK_Datasheet_Link"
-F 9 "/product-detail/en/te-connectivity-amp-connectors/640456-2/A1921-ND/109003" H 2100 6000 60  0001 L CNN "DK_Detail_Page"
-F 10 "CONN HEADER VERT 2POS 2.54MM" H 2100 6100 60  0001 L CNN "Description"
-F 11 "TE Connectivity AMP Connectors" H 2100 6200 60  0001 L CNN "Manufacturer"
-F 12 "Active" H 2100 6300 60  0001 L CNN "Status"
-	1    1900 5100
-	0    1    1    0
 $EndComp
 Wire Wire Line
@@
 Wire Wire Line
 	2350 5400 2350 5200
-Connection ~ 2350 5200
-Wire Wire Line
-	2350 5200 2000 5200
 Wire Wire Line
 	2350 5100 2350 4950
-Connection ~ 2350 5100
-Wire Wire Line
-	2350 5100 2000 5100
 Text Notes 5250 1650 0    50   ~ 0
 Make sure C6 is close to pin 44 of RP2040\n
@@
 Text Notes 800  6950 0    98   ~ 0
 Flash
+Text Label 5950 5250 0    50   ~ 0
+MIC_OUT
+Wire Wire Line
+	5100 5250 5950 5250
+$Comp
+L Connector_Generic:Conn_01x04 J?
+U 1 1 61FC5AD2
+P 1300 5200
+F 0 "J?" H 1218 4775 50  0000 C CNN
+F 1 "Conn_01x04" H 1218 4866 50  0000 C CNN
+F 2 "" H 1300 5200 50  0001 C CNN
+F 3 "~" H 1300 5200 50  0001 C CNN
+	1    1300 5200
+	-1   0    0    1
+$EndComp
+Connection ~ 2350 5100
+Wire Wire Line
+	1500 5100 2350 5100
+Wire Wire Line
+	2350 5200 1500 5200
+Connection ~ 2350 5200
+Wire Wire Line
+	1500 5300 1650 5300
+$Comp
+L power:GND #PWR?
+U 1 1 6212D0E2
+P 1650 5850
+F 0 "#PWR?" H 1650 5600 50  0001 C CNN
+F 1 "GND" H 1655 5677 50  0000 C CNN
+F 2 "" H 1650 5850 50  0001 C CNN
+F 3 "" H 1650 5850 50  0001 C CNN
+	1    1650 5850
+	1    0    0    -1
+$EndComp
+Wire Wire Line
+	1650 5300 1650 5850
+$Comp
+L power:+3V3 #PWR?
+U 1 1 62158E3F
+P 1850 4800
+F 0 "#PWR?" H 1850 4650 50  0001 C CNN
+F 1 "+3V3" H 1865 4973 50  0000 C CNN
+F 2 "" H 1850 4800 50  0001 C CNN
+F 3 "" H 1850 4800 50  0001 C CNN
+	1    1850 4800
+	1    0    0    -1
+$EndComp
+Wire Wire Line
+	1850 4800 1850 5000
+Wire Wire Line
+	1850 5000 1500 5000
 $EndSCHEMATC

Commit message: Update symbol ref
Parts:
- U3: symbol Memory_Flash:W25Q80DVSNIG -> mysymbols:W25Q80DVSNIG
Changed lines of the file:
@@
 	2600 5200 2350 5200
 $Comp
-L Memory_Flash:W25Q80DVSNIG U3
+L mysymbols:W25Q80DVSNIG U3
 U 1 1 616CDED3
 P 4300 8350

Commit message: Add transistor driver for leds
Parts:
- added D10, D11: LED, symbol Device:LED
- added Q1, Q10, Q11, Q2, Q3, Q4, Q5, Q6, Q7, Q8, Q9: 2N2222, digikey-footprints:TO-18-3, symbol dk_Transistors-Bipolar-BJT-Single:2N2222
- added R21, R22: 330, symbol Device:R
- added R23, R24, R25, R26, R27, R28, R29, R30, R31, R32, R33: 6.6k, symbol Device:R
- gave numbers to parts that had none: 1
Connections:
- wire segments 372 -> 431
Other:
- moved on the sheet: C15, C16, C17, C18, D1, MK1, R14, R15, R16, R17, R18, R19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
